Commit message: Reduce xacro argument count
* Remove unused xacro arguments specific to the ur_robot_driver

* Add robot model argument to automatically find the corresponding
configuration files for kinematics and visualisation

File: ur_description/urdf/ur.ros2_control.xacro (robot description, xacro)
@@ -3,10 +3,6 @@
   <xacro:macro name="ur_ros2_control" params="name prefix
     use_fake_hardware:=false fake_sensor_commands:=false
-    headless_mode:=false
     initial_positions:=${dict(shoulder_pan_joint=0.0,shoulder_lift_joint=-1.57,elbow_joint=0.0,wrist_1_joint=-1.57,wrist_2_joint=0.0,wrist_3_joint=0.0)}
-    use_tool_communication:=false
-    script_filename output_recipe_filename
-    input_recipe_filename tf_prefix
-    hash_kinematics robot_ip">
+    robot_ip">
     <ros2_control name="${name}" type="system">
       <hardware>
@@ -17,26 +13,6 @@
         </xacro:if>
         <xacro:unless value="${use_fake_hardware}">
-          <plugin>ur_robot_driver/URPositionHardwareInterface</plugin>
+          <plugin>robot_interface/universal_robots/UniversalRobotsInterface</plugin>
           <param name="robot_ip">${robot_ip}</param>
-          <param name="script_filename">${script_filename}</param>
-          <param name="output_recipe_filename">${output_recipe_filename}</param>
-          <param name="input_recipe_filename">${input_recipe_filename}</param>
-          <param name="headless_mode">${headless_mode}</param>
-          <param name="reverse_port">50001</param>
-          <param name="script_sender_port">50002</param>
-          <param name="tf_prefix">"${tf_prefix}"</param>
-          <param name="non_blocking_read">0</param>
-          <param name="servoj_gain">2000</param>
-          <param name="servoj_lookahead_time">0.03</param>
-          <param name="use_tool_communication">${use_tool_communication}</param>
-          <param name="kinematics/hash">"${hash_kinematics}"</param>
-          <param name="tool_voltage">0</param>
-          <param name="tool_parity">0</param>
-          <param name="tool_baud_rate">115200</param>
-          <param name="tool_stop_bits">1</param>
-          <param name="tool_rx_idle_chars">1.5</param>
-          <param name="tool_tx_idle_chars">3.5</param>
-          <param name="tool_device_name">/tmp/ttyUR</param>
-          <param name="tool_tcp_port">54321</param>
         </xacro:unless>
       </hardware>
@@ -133,110 +109,4 @@
         <state_interface name="torque.z"/>
       </sensor>
-      <!-- NOTE The following are joints used only for testing with fake hardware and will change in the future -->
-      <joint name="speed_scaling">
-        <state_interface name="speed_scaling_factor"/>
-        <param name="initial_speed_scaling_factor">1</param>
-        <command_interface name="target_speed_fraction_cmd"/>
-        <command_interface name="target_speed_fraction_async_success"/>
-      </joint>
-      <joint name="gpio">
-        <command_interface name="standard_digital_output_cmd_0"/>
-        <command_interface name="standard_digital_output_cmd_1"/>
-        <command_interface name="standard_digital_output_cmd_2"/>
-        <command_interface name="standard_digital_output_cmd_3"/>
-        <command_interface name="standard_digital_output_cmd_4"/>
-        <command_interface name="standard_digital_output_cmd_5"/>
-        <command_interface name="standard_digital_output_cmd_6"/>
-        <command_interface name="standard_digital_output_cmd_7"/>
-        <command_interface name="standard_digital_output_cmd_8"/>
-        <command_interface name="standard_digital_output_cmd_9"/>
-        <command_interface name="standard_digital_output_cmd_10"/>
-        <command_interface name="standard_digital_output_cmd_11"/>
-        <command_interface name="standard_digital_output_cmd_12"/>
-        <command_interface name="standard_digital_output_cmd_13"/>
-        <command_interface name="standard_digital_output_cmd_14"/>
-        <command_interface name="standard_digital_output_cmd_15"/>
-        <command_interface name="standard_digital_output_cmd_16"/>
-        <command_interface name="standard_digital_output_cmd_17"/>
-        <command_interface name="standard_analog_output_cmd_0"/>
-        <command_interface name="standard_analog_output_cmd_1"/>
-        <command_interface name="io_async_success"/>
-        <state_interface name="digital_output_0"/>
-        <state_interface name="digital_output_1"/>
-        <state_interface name="digital_output_2"/>
-        <state_interface name="digital_output_3"/>
-        <state_interface name="digital_output_4"/>
-        <state_interface name="digital_output_5"/>
-        <state_interface name="digital_output_6"/>
-        <state_interface name="digital_output_7"/>
-        <state_interface name="digital_output_8"/>
-        <state_interface name="digital_output_9"/>
-        <state_interface name="digital_output_10"/>
-        <state_interface name="digital_output_11"/>
-        <state_interface name="digital_output_12"/>
-        <state_interface name="digital_output_13"/>
-        <state_interface name="digital_output_14"/>
-        <state_interface name="digital_output_15"/>
-        <state_interface name="digital_output_16"/>
-        <state_interface name="digital_output_17"/>
-        <state_interface name="digital_input_0"/>
-        <state_interface name="digital_input_1"/>
-        <state_interface name="digital_input_2"/>
-        <state_interface name="digital_input_3"/>
-        <state_interface name="digital_input_4"/>
-        <state_interface name="digital_input_5"/>
-        <state_interface name="digital_input_6"/>
-        <state_interface name="digital_input_7"/>
-        <state_interface name="digital_input_8"/>
-        <state_interface name="digital_input_9"/>
-        <state_interface name="digital_input_10"/>
-        <state_interface name="digital_input_11"/>
-        <state_interface name="digital_input_12"/>
-        <state_interface name="digital_input_13"/>
-        <state_interface name="digital_input_14"/>
-        <state_interface name="digital_input_15"/>
-        <state_interface name="digital_input_16"/>
-        <state_interface name="digital_input_17"/>
-        <state_interface name="standard_analog_output_0"/>
-        <state_interface name="standard_analog_output_1"/>
-        <state_interface name="standard_analog_input_0"/>
-        <state_interface name="standard_analog_input_1"/>
-        <state_interface name="analog_io_type_0"/>
-        <state_interface name="analog_io_type_1"/>
-        <state_interface name="analog_io_type_2"/>
-        <state_interface name="analog_io_type_3"/>
-        <state_interface name="tool_mode"/>
-        <state_interface name="tool_output_voltage"/>
-        <state_interface name="tool_output_current"/>
-        <state_interface name="tool_temperature"/>
-        <state_interface name="tool_analog_input_0"/>
-        <state_interface name="tool_analog_input_1"/>
-        <state_interface name="tool_analog_input_type_0"/>
-        <state_interface name="tool_analog_input_type_1"/>
-        <state_interface name="robot_mode"/>
-        <state_interface name="robot_status_bit_0"/>
-        <state_interface name="robot_status_bit_1"/>
-        <state_interface name="robot_status_bit_2"/>
-        <state_interface name="robot_status_bit_3"/>
-        <state_interface name="safety_mode"/>
-        <state_interface name="safety_status_bit_0"/>
-        <state_interface name="safety_status_bit_1"/>
-        <state_interface name="safety_status_bit_2"/>
-        <state_interface name="safety_status_bit_3"/>
-        <state_interface name="safety_status_bit_4"/>
-        <state_interface name="safety_status_bit_5"/>
-        <state_interface name="safety_status_bit_6"/>
-        <state_interface name="safety_status_bit_7"/>
-        <state_interface name="safety_status_bit_8"/>
-        <state_interface name="safety_status_bit_9"/>
-        <state_interface name="safety_status_bit_10"/>
-      </joint>
-      <joint name="resend_robot_program">
-        <command_interface name="resend_robot_program_cmd"/>
-        <command_interface name="resend_robot_program_async_success"/>
-      </joint>
-      <joint name="system_interface">
-        <state_interface name="initialized"/>
-      </joint>
     </ros2_control>
   </xacro:macro>

File: ur_description/urdf/ur.urdf.xacro (robot description, xacro)
@@ -6,9 +6,6 @@
    <xacro:include filename="$(find ur_description)/urdf/ur_macro.xacro"/>
    <!-- parameters -->
-   <xacro:arg name="prefix" default="" />
-   <xacro:arg name="joint_limit_params" default=""/>
-   <xacro:arg name="kinematics_params" default=""/>
-   <xacro:arg name="physical_params" default=""/>
-   <xacro:arg name="visual_params" default=""/>
+   <xacro:arg name="model" default="ur5" />
+   <xacro:arg name="prefix" default="ur5_" />
    <xacro:arg name="transmission_hw_interface" default=""/>
    <xacro:arg name="safety_limits" default="false"/>
@@ -18,17 +15,14 @@
    <xacro:arg name="use_fake_hardware" default="false" />
    <xacro:arg name="fake_sensor_commands" default="false" />
-   <xacro:arg name="headless_mode" default="false" />
-   <xacro:arg name="use_tool_communication" default="false" />
-   <!-- initial position for fake hardware -->
-   <xacro:arg name="initial_positions_file" default="$(find ur_description)/config/initial_positions.yaml"/>
-   <!-- convert to property to use substitution in function -->
-   <xacro:property name="initial_positions_file" default="$(arg initial_positions_file)"/>
+   <!-- locate configuration files -->
+   <xacro:property name="initial_positions_file" default="$(find ur_description)/config/initial_positions.yaml"/>
+   <xacro:property name="model_config_path" default="$(find ur_description)/config/$(arg model)"/>
    <!-- arm -->
    <xacro:ur_robot
      prefix="$(arg prefix)"
-     joint_limits_parameters_file="$(arg joint_limit_params)"
-     kinematics_parameters_file="$(arg kinematics_params)"
-     physical_parameters_file="$(arg physical_params)"
-     visual_parameters_file="$(arg visual_params)"
+     joint_limits_parameters_file="${model_config_path}/joint_limits.yaml"
+     kinematics_parameters_file="${model_config_path}/default_kinematics.yaml"
+     physical_parameters_file="${model_config_path}/physical_parameters.yaml"
+     visual_parameters_file="${model_config_path}/visual_parameters.yaml"
      transmission_hw_interface="$(arg transmission_hw_interface)"
      safety_limits="$(arg safety_limits)"
@@ -37,6 +31,4 @@
      use_fake_hardware="$(arg use_fake_hardware)"
      fake_sensor_commands="$(arg fake_sensor_commands)"
-     headless_mode="$(arg headless_mode)"
-     initial_positions="${load_yaml(initial_positions_file)}"
-     use_tool_communication="$(arg use_tool_communication)" />
+     initial_positions="${load_yaml(initial_positions_file)}" />
 </robot>

File: ur_description/urdf/ur_macro.xacro (robot description, xacro)
@@ -56,7 +56,5 @@
     use_fake_hardware:=false
     fake_sensor_commands:=false
-    headless_mode:=false
-    initial_positions:=${dict(shoulder_pan_joint=0.0,shoulder_lift_joint=-1.57,elbow_joint=0.0,wrist_1_joint=-1.57,wrist_2_joint=0.0,wrist_3_joint=0.0)}
-    use_tool_communication:=false">
+    initial_positions:=${dict(shoulder_pan_joint=0.0,shoulder_lift_joint=-1.57,elbow_joint=0.0,wrist_1_joint=-1.57,wrist_2_joint=0.0,wrist_3_joint=0.0)}">
     <!-- Load configuration data from the provided .yaml files -->
     <xacro:read_model_data
@@ -66,7 +64,4 @@
       visual_parameters_file="${visual_parameters_file}"/>
     <!-- Data files required by the UR driver -->
-    <xacro:arg name="script_filename" default="$(find ur_robot_driver)/resources/ros_control.urscript"/>
-    <xacro:arg name="output_recipe_filename" default="$(find ur_robot_driver)/resources/rtde_output_recipe.txt"/>
-    <xacro:arg name="input_recipe_filename" default="$(find ur_robot_driver)/resources/rtde_input_recipe.txt"/>
     <xacro:arg name="robot_ip" default="10.0.1.186"/>
     <!-- ros2 control include -->
@@ -78,12 +73,5 @@
       initial_positions="${initial_positions}"
       fake_sensor_commands="$(arg fake_sensor_commands)"
-      headless_mode="$(arg headless_mode)"
-      script_filename="$(arg script_filename)"
-      output_recipe_filename="$(arg output_recipe_filename)"
-      input_recipe_filename="$(arg input_recipe_filename)"
-      tf_prefix=""
-      hash_kinematics="${kinematics_hash}"
-      robot_ip="$(arg robot_ip)"
-      use_tool_communication="$(arg use_tool_communication)"/>
+      robot_ip="$(arg robot_ip)"/>
     <!-- Add URDF transmission elements (for ros_control) -->
     <!--<xacro:ur_arm_transmission prefix="${prefix}" hw_interface="${transmission_hw_interface}" />-->
