Commit message: Add connected_to argument

File: ur_description/urdf/ur.urdf.xacro (robot description, xacro)
@@ -8,4 +8,5 @@
    <xacro:arg name="model" default="ur5" />
    <xacro:arg name="prefix" default="ur5_" />
+   <xacro:arg name="connected_to" default="" />
    <xacro:arg name="robot_ip" default="" />
    <xacro:arg name="transmission_hw_interface" default=""/>
@@ -23,4 +24,5 @@
      prefix="$(arg prefix)"
      robot_ip="$(arg robot_ip)"
+     connected_to="$(arg connected_to)"
      joint_limits_parameters_file="${model_config_path}/joint_limits.yaml"
      kinematics_parameters_file="${model_config_path}/default_kinematics.yaml"

File: ur_description/urdf/ur_macro.xacro (robot description, xacro)
@@ -46,4 +46,5 @@
   <xacro:macro name="ur_robot" params="
     prefix
+    connected_to:=''
     robot_ip
     joint_limits_parameters_file
@@ -76,6 +77,12 @@
     <!--<xacro:ur_arm_transmission prefix="${prefix}" hw_interface="${transmission_hw_interface}" />-->
     <!-- Placeholder for ros2_control transmission which don't yet exist -->
+    <xacro:if value="${connected_to == ''}">
+      <link name="world" />
+      <xacro:property name="base_frame_name" value="world"/>
+    </xacro:if>
+    <xacro:unless value="${connected_to == ''}">
+      <xacro:property name="base_frame_name" value="${connected_to}"/>
+    </xacro:unless>
     <!-- links -  main serial chain -->
-    <link name="${prefix}base_link"/>
     <link name="${prefix}base_link_inertia">
       <visual>
@@ -310,5 +317,5 @@
       -->
       <origin xyz="0 0 0" rpy="0 0 ${pi}"/>
-      <parent link="${prefix}base_link"/>
+      <parent link="${base_frame_name}"/>
       <child link="${prefix}base"/>
     </joint>
