Commit message: Fix urdf tree

File: ur_description/urdf/ur_macro.xacro (robot description, xacro)
@@ -227,5 +227,5 @@
     <!-- joints - main serial chain -->
     <joint name="${prefix}base_link-base_link_inertia" type="fixed">
-      <parent link="${prefix}base_link" />
+      <parent link="${base_frame_name}" />
       <child link="${prefix}base_link_inertia" />
       <!-- 'base_link' is REP-103 aligned (so X+ forward), while the internal

Commit message: Add connected_to to urdf and fix launch (#1)
* Remove old arguments from launch

* Add connected_to argument

* Fix urdf tree

* Change RViz config

File: ur_description/urdf/ur_macro.xacro (robot description, xacro)
@@ -46,4 +46,5 @@
   <xacro:macro name="ur_robot" params="
     prefix
+    connected_to:=''
     robot_ip
     joint_limits_parameters_file
@@ -76,6 +77,12 @@
     <!--<xacro:ur_arm_transmission prefix="${prefix}" hw_interface="${transmission_hw_interface}" />-->
     <!-- Placeholder for ros2_control transmission which don't yet exist -->
+    <xacro:if value="${connected_to == ''}">
+      <link name="world" />
+      <xacro:property name="base_frame_name" value="world"/>
+    </xacro:if>
+    <xacro:unless value="${connected_to == ''}">
+      <xacro:property name="base_frame_name" value="${connected_to}"/>
+    </xacro:unless>
     <!-- links -  main serial chain -->
-    <link name="${prefix}base_link"/>
     <link name="${prefix}base_link_inertia">
       <visual>
@@ -220,5 +227,5 @@
     <!-- joints - main serial chain -->
     <joint name="${prefix}base_link-base_link_inertia" type="fixed">
-      <parent link="${prefix}base_link" />
+      <parent link="${base_frame_name}" />
       <child link="${prefix}base_link_inertia" />
       <!-- 'base_link' is REP-103 aligned (so X+ forward), while the internal
@@ -310,5 +317,5 @@
       -->
       <origin xyz="0 0 0" rpy="0 0 ${pi}"/>
-      <parent link="${prefix}base_link"/>
+      <parent link="${base_frame_name}"/>
       <child link="${prefix}base"/>
     </joint>
