Commit message: Add adapter plate

File: ur_description/urdf/robotiq_hand_e_macro.xacro (robot description, xacro)
@@ -1,10 +1,10 @@
 <?xml version="1.0"?>
 <robot xmlns:xacro="http://wiki.ros.org/xacro">
-  <xacro:macro name="robotiq_e_hand" params="attached_to">
-    <link name="hand_base_link">
+  <xacro:macro name="robotiq_hand_e" params="attached_to">
+    <link name="adapter_link">
       <visual>
         <origin xyz="0 0 0" rpy="0 0 0"/>
         <geometry>
-          <mesh filename="package://ur_description/meshes/robotiq_hand_e/visual/robotiq_hand_e.dae"/>
+          <mesh filename="package://ur_description/meshes/robotiq/visual/adapter.dae" scale="0.001 0.001 0.001/>
         </geometry>
         <material name="Black">
@@ -15,12 +15,34 @@
         <origin xyz="0 0 0" rpy="0 0 0"/>
         <geometry>
-          <mesh filename="package://ur_description/meshes/robotiq_hand_e/visual/robotiq_hand_e.stl"/>
+          <mesh filename="package://ur_description/meshes/robotiq/visual/adapter.stl" scale="0.001 0.001 0.001/>
         </geometry>
       </collision>
     </link>
-    <joint name="${attached_to}_hand_joint" type="fixed">
+    <link name="hand_link">
+      <visual>
+        <origin xyz="0 0 0" rpy="0 0 0"/>
+        <geometry>
+          <mesh filename="package://ur_description/meshes/robotiq/visual/hand_e.dae" scale="0.001 0.001 0.001/>
+        </geometry>
+        <material name="Black">
+          <color rgba="0.0 0.0 0.0 1.0"/>
+        </material>
+      </visual>
+      <collision>
+        <origin xyz="0 0 0" rpy="0 0 0"/>
+        <geometry>
+          <mesh filename="package://ur_description/meshes/robotiq/visual/hand_e.stl" scale="0.001 0.001 0.001/>
+        </geometry>
+      </collision>
+    </link>
+    <joint name="${attached_to}_adapter_joint" type="fixed">
       <parent link="${attached_to}" />
-      <child link="hand_base_link" />
-      <origin xyz="0 0 0" rpy="0 0 0" />
+      <child link="adapter_link" />
+      <origin xyz="0 0 0" rpy="1.57 0 1.57" />
+    </joint>
+    <joint name="adapter_hand_joint" type="fixed">
+      <parent link="adapter_link />
+      <child link="hand_link" />
+      <origin xyz="0 0 0.1" rpy="0 0 0" />
     </joint>
   </xacro:macro>

File: ur_description/urdf/ur.urdf.xacro (robot description, xacro)
@@ -5,4 +5,5 @@
    <!-- import main macro -->
    <xacro:include filename="$(find ur_description)/urdf/ur_macro.xacro"/>
+   <xacro:include filename="$(find ur_description)/urdf/robotiq_hand_e_macro.xacro"/>
    <!-- parameters -->
    <xacro:arg name="model" default="ur5" />
@@ -19,5 +20,5 @@
    <xacro:arg name="use_tcp_fts_sensor" default="false" />
    <xacro:arg name="fake_sensor_commands" default="false" />
-   <xacro:arg name="robotiq_hand_e" default="false= />
+   <xacro:arg name="robotiq_hand_e" default="false" />
    <!-- locate configuration files -->
    <xacro:property name="initial_positions_file" default="$(find ur_description)/config/initial_positions.yaml"/>
@@ -40,6 +41,6 @@
      fake_sensor_commands="$(arg fake_sensor_commands)"
      initial_positions="${load_yaml(initial_positions_file)}" />
-   <xacro:if value="${robotiq_hand_e}">
-     <xacro:robotiq_hand_e attached_to:="${prefix}tool0" />
+   <xacro:if value="$(arg robotiq_hand_e)">
+     <xacro:robotiq_hand_e attached_to="$(arg prefix)tool0" />
    </xacro:if>
 </robot>

Commit message: Fixes and better tfs

File: ur_description/urdf/robotiq_hand_e_macro.xacro (robot description, xacro)
@@ -6,8 +6,8 @@
         <origin xyz="0 0 0" rpy="0 0 0"/>
         <geometry>
-          <mesh filename="package://ur_description/meshes/robotiq/visual/adapter.dae" scale="0.001 0.001 0.001/>
+          <mesh filename="package://ur_description/meshes/robotiq/collision/adapter.stl" scale="0.001 0.001 0.001"/>
         </geometry>
-        <material name="Black">
-          <color rgba="0.0 0.0 0.0 1.0"/>
+        <material name="AlmostBlack">
+          <color rgba="0.1 0.1 0.1 1.0"/>
         </material>
       </visual>
@@ -15,5 +15,5 @@
         <origin xyz="0 0 0" rpy="0 0 0"/>
         <geometry>
-          <mesh filename="package://ur_description/meshes/robotiq/visual/adapter.stl" scale="0.001 0.001 0.001/>
+          <mesh filename="package://ur_description/meshes/robotiq/collision/adapter.stl" scale="0.001 0.001 0.001"/>
         </geometry>
       </collision>
@@ -23,8 +23,8 @@
         <origin xyz="0 0 0" rpy="0 0 0"/>
         <geometry>
-          <mesh filename="package://ur_description/meshes/robotiq/visual/hand_e.dae" scale="0.001 0.001 0.001/>
+          <mesh filename="package://ur_description/meshes/robotiq/collision/hand_e.stl" scale="0.001 0.001 0.001"/>
         </geometry>
-        <material name="Black">
-          <color rgba="0.0 0.0 0.0 1.0"/>
+        <material name="AlmostBlack">
+          <color rgba="0.1 0.1 0.1 1.0"/>
         </material>
       </visual>
@@ -32,17 +32,23 @@
         <origin xyz="0 0 0" rpy="0 0 0"/>
         <geometry>
-          <mesh filename="package://ur_description/meshes/robotiq/visual/hand_e.stl" scale="0.001 0.001 0.001/>
+          <mesh filename="package://ur_description/meshes/robotiq/collision/hand_e.stl" scale="0.001 0.001 0.001"/>
         </geometry>
       </collision>
     </link>
+    <link name="fingers_link"/>
     <joint name="${attached_to}_adapter_joint" type="fixed">
       <parent link="${attached_to}" />
       <child link="adapter_link" />
-      <origin xyz="0 0 0" rpy="1.57 0 1.57" />
+      <origin rpy="0 0 -1.57" xyz="0 0 0.005"/>
     </joint>
     <joint name="adapter_hand_joint" type="fixed">
-      <parent link="adapter_link />
+      <parent link="adapter_link" />
       <child link="hand_link" />
-      <origin xyz="0 0 0.1" rpy="0 0 0" />
+      <origin xyz="0 0 0.1" rpy="0 0 0.093" />
+    </joint>
+    <joint name="hand_finger_joint" type="fixed">
+      <parent link="hand_link"/>
+      <child link="fingers_link"/>
+      <origin rpy="-1.57 0 0" xyz="0 0.06 0"/>
     </joint>
   </xacro:macro>

Commit message: Final updates

File: ur_description/urdf/robotiq_hand_e_macro.xacro (robot description, xacro)
@@ -19,5 +19,5 @@
       </collision>
     </link>
-    <link name="hand_link">
+    <link name="robotiq_hand_e">
       <visual>
         <origin xyz="0 0 0" rpy="0 0 0"/>
@@ -36,19 +36,19 @@
       </collision>
     </link>
-    <link name="fingers_link"/>
+    <link name="fingertip"/>
     <joint name="${attached_to}_adapter_joint" type="fixed">
       <parent link="${attached_to}" />
       <child link="adapter_link" />
-      <origin rpy="0 0 -1.57" xyz="0 0 0.005"/>
+      <origin rpy="0 0 -1.57" xyz="0 0 0.006" />
     </joint>
     <joint name="adapter_hand_joint" type="fixed">
       <parent link="adapter_link" />
-      <child link="hand_link" />
-      <origin xyz="0 0 0.1" rpy="0 0 0.093" />
+      <child link="robotiq_hand_e" />
+      <origin rpy="1.57 0 0" xyz="0 0 0.094" />
     </joint>
     <joint name="hand_finger_joint" type="fixed">
-      <parent link="hand_link"/>
-      <child link="fingers_link"/>
-      <origin rpy="-1.57 0 0" xyz="0 0.06 0"/>
+      <parent link="robotiq_hand_e" />
+      <child link="fingertip" />
+      <origin rpy="-1.57 1.57 0" xyz="0 0.06 0" />
     </joint>
   </xacro:macro>
